File: rfd77101-bat-powered/power_mgmt.sch (KiCad schematic (older format))
At the start: 16 parts, among them J1 USB_OTG, J2 BATT_CONN, Q1 Q_NMOS_GSD, Q2 Q_PMOS_GSD, U2 MCP73811T-420I-OT, U3 TLV74130

Commit message: update board for better batt measurements
Parts:
- removed R5: 1.6k, Resistor_SMD:R_0603_1608Metric, symbol R
- added Q3: DMP3099L-13, Package_TO_SOT_SMD:SOT-23, symbol Device:Q_PMOS_GSD
- added R5: 10k, Resistor_SMD:R_0603_1608Metric, symbol Device:R
- C1, C2, C3, C4: symbol C -> Device:C
- D1, D2: symbol D_Schottky -> Device:D_Schottky
- J1: value USB_OTG -> USB_B_Micro; symbol USB_OTG -> Connector_Specialized:USB_B_Micro
- J2: symbol CONN_01X02 -> Connector_Generic:Conn_01x02
- Q1: symbol Q_NMOS_GSD -> Device:Q_NMOS_GSD
- Q2: value Q_PMOS_GSD -> DMP3099L-13; symbol Q_PMOS_GSD -> Device:Q_PMOS_GSD
- R1: value 1.6k -> 3.1k; symbol R -> Device:R
- R2, R3: symbol R -> Device:R
- U2: symbol MCP73811T-420I-OT -> Battery_Management:MCP73811T-420I-OT
- U3: symbol AP2204K-3.0 -> Regulator_Linear:AP2204K-3.0
Connections:
- net +BATT: now also Q3.2 (S), R5.1
- net GND: now also R2.2
- net at R1.1: now also Q3.3 (D)
- net at Q1.3 (D): now also Q3.1 (G), R5.2; no longer R2.2
Other:
- moved on the sheet: Q1, R1, R2
