File: rfd77101-bat-powered/rfd77101-bat-powered.sch (KiCad schematic (older format))
At the start: 5 parts, among them J3 Conn_01x07, U1 RFD77101

Commit message: update board for better batt measurements
Parts:
- C5: symbol C -> Device:C
- D3: symbol LED -> Device:LED
- J3: symbol Conn_01x07 -> Connector_Generic:Conn_01x07
- R4: symbol R -> Device:R
- U1: symbol RFD77101 -> RF_Bluetooth:RFD77101
Changed lines of the file:
@@
-EESchema Schematic File Version 2
-LIBS:power
-LIBS:device
-LIBS:transistors
-LIBS:conn
-LIBS:linear
-LIBS:regul
-LIBS:74xx
-LIBS:cmos4000
-LIBS:adc-dac
-LIBS:memory
-LIBS:xilinx
-LIBS:microcontrollers
-LIBS:dsp
-LIBS:microchip
-LIBS:analog_switches
-LIBS:motorola
-LIBS:texas
-LIBS:intel
-LIBS:audio
-LIBS:interface
-LIBS:digital-audio
-LIBS:philips
-LIBS:display
-LIBS:cypress
-LIBS:siliconi
-LIBS:opto
-LIBS:atmel
-LIBS:contrib
-LIBS:valves
-LIBS:RF_Bluetooth
-LIBS:Battery_Management
+EESchema Schematic File Version 4
 LIBS:rfd77101-bat-powered-cache
-EELAYER 25 0
+EELAYER 26 0
 EELAYER END
 $Descr A4 11693 8268
@@
 $EndSheet
 $Comp
-L RFD77101 U1
+L RF_Bluetooth:RFD77101 U1
 U 1 1 5A93FA36
 P 8050 3250
@@
 $EndComp
 $Comp
-L Conn_01x07 J3
+L Connector_Generic:Conn_01x07 J3
 U 1 1 5A940680
 P 3300 1600
@@
 SWDIO/RESET
 $Comp
-L GND #PWR01
+L power:GND #PWR01
 U 1 1 5A94075B
 P 3650 2000
@@
 $EndComp
 $Comp
-L VBUS #PWR02
+L power:VBUS #PWR02
 U 1 1 5A94077F
 P 4250 1450
@@
 BATT_V_EN
 $Comp
-L GND #PWR03
+L power:GND #PWR03
 U 1 1 5A942B55
 P 7950 5000
@@
 	7550 4550 7550 4800
 Wire Wire Line
-	7550 4800 8450 4800
-Wire Wire Line
-	7950 4550 7950 5000
+	7550 4800 7650 4800
+Wire Wire Line
+	7950 4550 7950 4800
 Wire Wire Line
 	7650 4550 7650 4800
@@
 Connection ~ 8350 4800
 $Comp
-L VDD #PWR04
+L power:VDD #PWR04
 U 1 1 5A942CC9
 P 8050 1800
@@
 	8050 1800 8050 1950
 $Comp
-L C C5
+L Device:C C5
 U 1 1 5A942D56
 P 5000 1650
@@
 $EndComp
 $Comp
-L VDD #PWR05
+L power:VDD #PWR05
 U 1 1 5A942E08
 P 5000 1350
@@
 $EndComp
 $Comp
-L GND #PWR06
+L power:GND #PWR06
 U 1 1 5A942E28
 P 5000 1950
@@
 	5000 1500 5000 1350
 $Comp
-L LED D3
+L Device:LED D3
 U 1 1 5A942EE5
 P 6200 1550
@@
 $EndComp
 $Comp
-L R R4
+L Device:R R4
 U 1 1 5A942F32
 P 6200 1950
@@
 $EndComp
 $Comp
-L GND #PWR07
+L power:GND #PWR07
 U 1 1 5A942F66
 P 6200 2200
@@
 Text Label 8750 3250 0    60   ~ 0
 LED_1
+Wire Wire Line
+	7650 4800 7750 4800
+Wire Wire Line
+	7750 4800 7850 4800
+Wire Wire Line
+	7850 4800 7950 4800
+Wire Wire Line
+	7950 4800 7950 5000
+Wire Wire Line
+	7950 4800 8050 4800
+Wire Wire Line
+	8050 4800 8150 4800
+Wire Wire Line
+	8150 4800 8250 4800
+Wire Wire Line
+	8250 4800 8350 4800
+Wire Wire Line
+	8350 4800 8450 4800
 $EndSCHEMATC
